File: hardware/kicad/balsun.kicad_pcb (KiCad board)
At the start: 4 copper layers, 64.4 x 53.3 mm, 83 parts, among them IC1 R7FA4M1AB3CFM#AA0, IC2 BP35C5, IC3 BP5293-50, IC4 XCL103D503CR-G, IC5 TPS2115APW, IC6 TPS2115APW, J1 HPH2-A-10-UA, J2 61301611821, J4 61301611821, J5 CX90B2-24P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

Commit message: update pattern
Parts:
- added REF**: phi1_pad, SamacSys_Parts:phi1_pad, F.Cu at (164.9, 76.5)
- added REF**: phi1_pad, SamacSys_Parts:phi1_pad, F.Cu at (218.8, 124.6)
Routing:
- net +5V: track 222.1 -> 225.7 mm
- net Net-(IC5-OUT): track 15.3 -> 18.2 mm
- net +3V3: track 96.1 -> 98.3 mm, vias 4 -> 3
- net P109_SCI9_TXD: track 14.9 -> 16.7 mm
- net Net-(IC3-OUT): track 16.8 -> 18.5 mm
- net WISUN_RX_Serial1_D1: track 36.1 -> 37.6 mm
- net GND: track 52.8 -> 53.9 mm
- net P015: track 21.2 -> 20.2 mm
- net P108_SWDIO: track 29.7 -> 28.8 mm
- net RESET: track 89.3 -> 88.5 mm
- net P111_GPT3_A: track 51.9 -> 52.4 mm
Other:
- board text added: ".."
- board text added: "Balsun"
- board text added: "ver.1"
- board text removed: "1k"
